Commit message: turn the wrist from fixed to revolute(F)

File: Robots/talos/talos_reduced_armfixed.urdf (robot description, URDF)
Before this commit: robot talos, 60 links, 59 joints
Joints:
- joint wrist_right_ft_joint: axis (none) -> 0 0 1; limit (none) -> lower=-1.57 upper=1.57 effort=10.0 velocity=1.0; type fixed -> revolute

File: Robots/talos/talos_reduced_armfixed_floatingbase.urdf (robot description, URDF)
Before this commit: robot talos, 66 links, 65 joints
Joints:
- joint wrist_right_ft_joint: axis (none) -> 0 0 1; limit (none) -> lower=-1.57 upper=1.57 effort=10.0 velocity=1.0; origin xyz=0 0 -0.051 rpy=0.0 0 -1.57079632679 -> xyz=0 0 -0.051 rpy=0.0 0 -4.71238898038314; type fixed -> revolute

Commit message: q

File: Robots/talos/talos_reduced_armfixed.urdf (robot description, URDF)
Before this commit: robot talos, 60 links, 59 joints
Joints:
- joint arm_right_1_joint: origin xyz=0.00000 -0.1575 0.23200 rpy=0.0 0.0 0.0 -> xyz=0.00000 -0.1575 0.23200 rpy=0.0 -1.57 0.0; type fixed -> revolute
- joint arm_right_4_joint: origin xyz=0.02000 0.00000 -0.27300 rpy=0.0 0.0 0.0 -> xyz=0.02000 0.00000 -0.27300 rpy=0.0 -1.57 0.0
- joint arm_right_6_joint: origin xyz=0.00000 0.00000 0.00000 rpy=0.0 0.0 0.0 -> xyz=0.00000 0.00000 0.0 rpy=0.0 0.0 0.0
- joint arm_right_7_joint: origin xyz=0.0 0.0 0.0 rpy=0.0 0.0 0.0 -> xyz=0.0 0.0 0.0 rpy=0.0 -1.57 0.0
- joint wrist_right_ft_joint: axis 0 0 1 -> (none); limit lower=-1.57 upper=1.57 effort=10.0 velocity=1.0 -> (none); type revolute -> fixed

File: Robots/talos/talos_reduced_armfixed_floatingbase.urdf (robot description, URDF)
Before this commit: robot talos, 66 links, 65 joints
Joints:
- joint arm_right_1_joint: origin xyz=0.00000 -0.1575 0.23200 rpy=0.0 0.0 0.0 -> xyz=0.00000 -0.1575 0.23200 rpy=0.0 -1.57 0.0; type fixed -> revolute
- joint arm_right_7_joint: origin xyz=0.0 0.0 0.0 rpy=0.0 0.0 0.0 -> xyz=0.0 0.0 0.0 rpy=0.0 -1.57 0.0
- joint wrist_right_ft_joint: axis 0 0 1 -> (none); limit lower=-1.57 upper=1.57 effort=10.0 velocity=1.0 -> (none); type revolute -> fixed

Commit message: fail test

File: Robots/talos/talos_reduced_armfixed.urdf (robot description, URDF)
Before this commit: robot talos, 60 links, 59 joints
Joints:
- joint arm_right_1_joint: origin xyz=0.00000 -0.1575 0.23200 rpy=0.0 0.0 0.0 -> xyz=0.00000 -0.1575 0.23200 rpy=0.0 -1.57 0.0; type fixed -> revolute

File: Robots/talos/talos_reduced_armfixed_floatingbase.urdf (robot description, URDF)
Before this commit: robot talos, 66 links, 65 joints
Joints:
- joint arm_right_1_joint: origin xyz=0.00000 -0.1575 0.23200 rpy=0.0 0.0 0.0 -> xyz=0.00000 -0.1575 0.23200 rpy=0.0 -1.57 0.0; type fixed -> revolute
